File: WordClock_GE423/word_clock.sch (EAGLE design)
At the start: 27 parts

Commit message: initial board
finished initial schematic
laid out (no routing) first board
Parts:
- removed U$2, U$3: SHIFT_REGISTER, word_clock:SHIFT_REGISTER
- added C1: 1u, rcl:C-US050-025X075
- added C2: 4.7u, rcl:C-US050-025X075
- added C3: 10u, rcl:C-US050-025X075
- added JP10, JP4, JP5, JP6, JP7, JP8, JP9: (no value), SparkFun-Connectors:M03-SCREW-5MM
- added Q1: 32.768kHz, crystal:CRYSTALTC26V
- added R1, R2, R3: 4.7k, rcl:R-US_0207/10
- added SERVO_1, SERVO_2: (no value), pinhead:PINHD-1X3
- added SR_1, SR_2: SHIFT_REGISTER, word_clock:SHIFT_REGISTER
- added U$27: FET, word_clock:FET
- added U$28: COIN_CELL_SPARKFUN, eoh:COIN_CELL_SPARKFUN
Connections:
- removed net JACK_PWR: JP1.PWR, U$4.VIN
- removed net N$3: U$10.G, U$11.G, U$12.G, U$13.G, U$14.G, U$15.G, U$16.G, U$17.G, U$18.G, U$19.G, U$20.G, U$21.G, U$22.G, U$23.G, U$24.G, U$5.G, U$6.G, U$7.G, U$8.G, U$9.G
- removed net VCC: U$1.A1, U$1.RST, U$1.VCC, U$2.A1, U$2.RST, U$2.VCC, U$3.A1, U$3.RST, U$3.VCC, U$4.VOUT
- new net 3.3V: C1.1, C3.1, R1.2, R2.2, R3.2, SR_1.A1, SR_1.RST, SR_1.VCC, SR_2.A1, SR_2.RST, SR_2.VCC, U$1.A1, U$1.RST, U$1.VCC, U$25.VCC, U$26.VCC, U$4.VOUT
- new net EIGHT: U$1.Q2, U$20.G
- new net EIGHT_LED: JP9.2, U$20.D
- new net ELEVEN: U$1.Q5, U$23.G
- new net ELEVEN_LED: JP10.2, U$23.D
- new net FIVE_HR: SR_2.Q6, U$17.G
- new net FIVE_HR_LED: JP8.2, U$17.D
- new net FIVE_MIN: SR_1.Q2, U$6.G
- new net FIVE_MIN_LED: JP4.3, U$6.D
- new net FOUR: SR_2.Q5, U$16.G
- new net FOUR_LED: JP8.1, U$16.D
- new net HALF: SR_1.Q6, U$10.G
- new net HALF_LED: JP6.1, U$10.D
- new net IRQ: R3.1, U$26.IRQ
- new net IT_IS: SR_1.Q1, U$5.G
- new net IT_IS_LED: JP4.1, U$5.D
- new net N$1: Q1.1, U$26.OSCO
- new net N$7: U$1.Q8
- new net NINE: U$1.Q3, U$21.G
- new net NINE_LED: JP9.3, U$21.D
- new net OCLK: U$1.Q7, U$27.G
- new net OCLK_LED: JP4.2, U$27.D
- new net ONE: SR_2.Q2, U$13.G
- new net ONE_LED: JP7.1, U$13.D
- new net PAST: SR_1.Q7, U$11.G
- new net PAST_LED: JP6.2, U$11.D
- new net QUARTER: SR_1.Q4, U$8.G
- new net QUARTER_LED: JP5.2, U$8.D
- new net RTC_SCL: R1.1, U$25.P1.6, U$26.SCL
- new net RTC_SDA: R2.1, U$25.P1.7, U$26.SDA
- new net SERVO_1: SERVO_1.2, U$25.P2.2
- new net SERVO_2: SERVO_2.2, U$25.P2.4
- new net SEVEN: U$1.Q1, U$19.G
- new net SEVEN_LED: JP9.1, U$19.D
- new net SIX: SR_2.Q7, U$18.G
- new net SIX_LED: JP8.3, U$18.D
- new net TEN_HR: U$1.Q4, U$22.G
- new net TEN_HR_LED: JP10.1, U$22.D
- new net TEN_MIN: SR_1.Q3, U$7.G
- new net TEN_MIN_LED: JP5.1, U$7.D
- new net THREE: SR_2.Q4, U$15.G
- new net THREE_LED: JP7.3, U$15.D
- new net TO: SR_2.Q1, U$12.G
- new net TO_LED: JP6.3, U$12.D
- new net TWELVE: U$1.Q6, U$24.G
- new net TWELVE_LED: JP10.3, U$24.D
- new net TWENTY: SR_1.Q5, U$9.G
- new net TWENTY_LED: JP5.3, U$9.D
- new net TWO: SR_2.Q3, U$14.G
- new net TWO_LED: JP7.2, U$14.D
- new net VBACK: U$26.VBACK, U$28.VDD_1, U$28.VDD_2
- new net VCC_5: C2.1, JP1.PWR, SERVO_1.1, SERVO_2.1, U$4.VIN
- net GND: now also C1.2, C2.2, C3.2, SERVO_1.3, SERVO_2.3, SR_1.GND, SR_2.GND, U$25.GND, U$26.GND, U$27.S, U$28.GND; no longer U$2.GND, U$3.GND
- net N$2: now also Q1.2, U$26.OSCI; no longer U$10.D, U$11.D, U$12.D, U$13.D, U$14.D, U$15.D, U$16.D, U$17.D, U$18.D, U$19.D, U$20.D, U$21.D, U$22.D, U$23.D, U$24.D, U$5.D, U$6.D, U$7.D, U$8.D, U$9.D
- net N$4: now also SR_1.Q8, SR_2.A2; no longer U$2.A2, U$3.Q8
- net N$5: now also SR_2.Q8; no longer U$2.Q8
- net SR_CLK: now also SR_1.CLK, SR_2.CLK, U$25.P1.0; no longer U$2.CLK, U$3.CLK
- net SR_DATA: now also SR_1.A2, U$25.P1.1; no longer U$3.A2
Other:
- moved on the sheet: JP1

Commit message: finished boards
finally. added VCC rail for LEDs
Parts:
- added LED_PWR: (no value), SparkFun-Connectors:M03-SCREW-5MM
- renumbered U$10 to 30M, U$11 to PAST, U$12 to TO, U$13 to 1H, U$14 to 2H, U$15 to 3H, U$16 to 4H, U$17 to 5H, U$18 to 6H, U$19 to 7H, U$20 to 8H, U$21 to 9H, U$22 to 10H, U$23 to 11H, U$24 to 12H, U$26 to RTC, U$27 to OCLK, U$5 to ITIS, U$6 to 5M, U$7 to 10M, U$8 to 15M, U$9 to 20M
Connections:
- net 3.3V: now also LED_PWR.1, LED_PWR.2, LED_PWR.3
